File: Duet-MainPCB/Duet-Switch-Tester.kicad_sch (KiCad schematic)
At the start: 37 parts, among them SW1 SW_Push, SW2 SW_Push, U1 ZD25Q80BNIGR, U2 PRTR5V0U2X, U3 RP2040, U4 AP7313-33SRG-7, Y1 12MHz

Commit message: Route PCB
Parts:
- C7: value Optional-Bulk -> 10uF-OPT
- R2: value 10k-Opt -> 10k-OPT
Connections:
- net COL0: now also U3.41 (GPIO29_ADC3); no longer U3.8 (GPIO6)
- net COL1: now also U3.40 (GPIO28_ADC2); no longer U3.9 (GPIO7)
- net COL10: now also U3.16 (GPIO13); no longer U3.27 (GPIO16)
- net COL11: now also U3.15 (GPIO12); no longer U3.28 (GPIO17)
- net COL12: now also U3.14 (GPIO11); no longer U3.29 (GPIO18)
- net COL13: now also U3.13 (GPIO10); no longer U3.30 (GPIO19)
- net COL14: now also U3.12 (GPIO9); no longer U3.31 (GPIO20)
- net COL15: now also U3.11 (GPIO8); no longer U3.32 (GPIO21)
- net COL16: now also U3.9 (GPIO7); no longer U3.34 (GPIO22)
- net COL17: now also U3.8 (GPIO6); no longer U3.35 (GPIO23)
- net COL2: now also U3.39 (GPIO27_ADC1); no longer U3.11 (GPIO8)
- net COL3: now also U3.38 (GPIO26_ADC0); no longer U3.12 (GPIO9)
- net COL4: now also U3.37 (GPIO25); no longer U3.13 (GPIO10)
- net COL5: now also U3.36 (GPIO24); no longer U3.14 (GPIO11)
- net COL6: now also U3.35 (GPIO23); no longer U3.15 (GPIO12)
- net COL7: now also U3.34 (GPIO22); no longer U3.16 (GPIO13)
- net COL8: now also U3.29 (GPIO18); no longer U3.17 (GPIO14)
- net COL9: now also U3.17 (GPIO14); no longer U3.18 (GPIO15)
