File: Duet-MainPCB/matrix.kicad_sch (KiCad schematic)
At the start: 216 parts, among them K1 CPG151101S11-16, K10 CPG151101S11-16, K100 CPG151101S11-16, K101 CPG151101S11-16, K102 CPG151101S11-16, K103 CPG151101S11-16, K104 CPG151101S11-16, K105 CPG151101S11-16, K106 CPG151101S11-16, K107 CPG151101S11-16, K108 CPG151101S11-16, K11 CPG151101S11-16, K12 CPG151101S11-16, K13 CPG151101S11-16, K14 CPG151101S11-16, K15 CPG151101S11-16, K16 CPG151101S11-16, K17 CPG151101S11-16, K18 CPG151101S11-16, K19 CPG151101S11-16, K2 CPG151101S11-16, K20 CPG151101S11-16, K21 CPG151101S11-16, K22 CPG151101S11-16, K23 CPG151101S11-16, K24 CPG151101S11-16, K25 CPG151101S11-16, K26 CPG151101S11-16, K27 CPG151101S11-16, K28 CPG151101S11-16, K29 CPG151101S11-16, K3 CPG151101S11-16, K30 CPG151101S11-16, K31 CPG151101S11-16, K32 CPG151101S11-16, K33 CPG151101S11-16, K34 CPG151101S11-16, K35 CPG151101S11-16, K36 CPG151101S11-16, K37 CPG151101S11-16, K38 CPG151101S11-16, K39 CPG151101S11-16, K4 CPG151101S11-16, K40 CPG151101S11-16, K41 CPG151101S11-16, K42 CPG151101S11-16, K43 CPG151101S11-16, K44 CPG151101S11-16, K45 CPG151101S11-16, K46 CPG151101S11-16, K47 CPG151101S11-16, K48 CPG151101S11-16, K49 CPG151101S11-16, K5 CPG151101S11-16, K50 CPG151101S11-16, K51 CPG151101S11-16, K52 CPG151101S11-16, K53 CPG151101S11-16, K54 CPG151101S11-16, K55 CPG151101S11-16, K56 CPG151101S11-16, K57 CPG151101S11-16, K58 CPG151101S11-16, K59 CPG151101S11-16, K6 CPG151101S11-16, K60 CPG151101S11-16, K61 CPG151101S11-16, K62 CPG151101S11-16, K63 CPG151101S11-16, K64 CPG151101S11-16, K65 CPG151101S11-16, K66 CPG151101S11-16, K67 CPG151101S11-16, K68 CPG151101S11-16, K69 CPG151101S11-16, K7 CPG151101S11-16, K70 CPG151101S11-16, K71 CPG151101S11-16, K72 CPG151101S11-16, K73 CPG151101S11-16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

Commit message: Route PCB
Parts:
- D1, D10, D100, D101, D102, D103, D104, D105, D106, D107, D108, D11, D12, D13, D14, D15, D16, D17, D18, D19, D2, D20, D21, D22, D23, D24, D25, D26, D27, D28, D29, D3, D30, D31, D32, D33, D34, D35, D36, D37, D38, D39, D4, D40, D41, D42, D43, D44, D45, D46, D47, D48, D49, D5, D50, D51, D52, D53, D54, D55, D56, D57, D58, D59, D6, D60, D61, D62, D63, D64, D65, D66, D67, D68, D69, D7, D70, D71, D72, D73, D74, D75, D76, D77, D78, D79, D8, D80, D81, D82, D83, D84, D85, D86, D87, D88, D89, D9, D90, D91, D92, D93, D94, D95, D96, D97, D98, D99: footprint Diode_SMD:D_SOD-123 -> locallib:D_SOD-123-MinimalPrint
Connections:
- net COL0: now also K1.1, K2.1, K3.1, K4.1, K5.1, K6.1; no longer K1.2, K2.2, K3.2, K4.2, K5.2, K6.2
- net COL1: now also K10.1, K11.1, K12.1, K7.1, K8.1, K9.1; no longer K10.2, K11.2, K12.2, K7.2, K8.2, K9.2
- net COL10: now also K61.1, K62.1, K63.1, K64.1, K65.1, K66.1; no longer K61.2, K62.2, K63.2, K64.2, K65.2, K66.2
- net COL11: now also K67.1, K68.1, K69.1, K70.1, K71.1, K72.1; no longer K67.2, K68.2, K69.2, K70.2, K71.2, K72.2
- net COL12: now also K73.1, K74.1, K75.1, K76.1, K77.1, K78.1; no longer K73.2, K74.2, K75.2, K76.2, K77.2, K78.2
- net COL13: now also K79.1, K80.1, K81.1, K82.1, K83.1, K84.1; no longer K79.2, K80.2, K81.2, K82.2, K83.2, K84.2
- net COL14: now also K85.1, K86.1, K87.1, K88.1, K89.1, K90.1; no longer K85.2, K86.2, K87.2, K88.2, K89.2, K90.2
- net COL15: now also K91.1, K92.1, K93.1, K94.1, K95.1, K96.1; no longer K91.2, K92.2, K93.2, K94.2, K95.2, K96.2
- net COL16: now also K100.1, K101.1, K102.1, K97.1, K98.1, K99.1; no longer K100.2, K101.2, K102.2, K97.2, K98.2, K99.2
- net COL17: now also K103.1, K104.1, K105.1, K106.1, K107.1, K108.1; no longer K103.2, K104.2, K105.2, K106.2, K107.2, K108.2
- net COL2: now also K13.1, K14.1, K15.1, K16.1, K17.1, K18.1; no longer K13.2, K14.2, K15.2, K16.2, K17.2, K18.2
- net COL3: now also K19.1, K20.1, K21.1, K22.1, K23.1, K24.1; no longer K19.2, K20.2, K21.2, K22.2, K23.2, K24.2
- net COL4: now also K25.1, K26.1, K27.1, K28.1, K29.1, K30.1; no longer K25.2, K26.2, K27.2, K28.2, K29.2, K30.2
- net COL5: now also K31.1, K32.1, K33.1, K34.1, K35.1, K36.1; no longer K31.2, K32.2, K33.2, K34.2, K35.2, K36.2
- net COL6: now also K37.1, K38.1, K39.1, K40.1, K41.1, K42.1; no longer K37.2, K38.2, K39.2, K40.2, K41.2, K42.2
- net COL7: now also K43.1, K44.1, K45.1, K46.1, K47.1, K48.1; no longer K43.2, K44.2, K45.2, K46.2, K47.2, K48.2
- net COL8: now also K49.1, K50.1, K51.1, K52.1, K53.1, K54.1; no longer K49.2, K50.2, K51.2, K52.2, K53.2, K54.2
- net COL9: now also K55.1, K56.1, K57.1, K58.1, K59.1, K60.1; no longer K55.2, K56.2, K57.2, K58.2, K59.2, K60.2
- net at D89.2 (A): now also K89.2; no longer K89.1
- net at D99.2 (A): now also K99.2; no longer K99.1
- net at D63.2 (A): now also K63.2; no longer K63.1
- net at D91.2 (A): now also K91.2; no longer K91.1
- net at D75.2 (A): now also K75.2; no longer K75.1
- net at D101.2 (A): now also K101.2; no longer K101.1
- net at D3.2 (A): now also K3.2; no longer K3.1
- net at D38.2 (A): now also K38.2; no longer K38.1
- net at D8.2 (A): now also K8.2; no longer K8.1
- net at D71.2 (A): now also K71.2; no longer K71.1
- net at D62.2 (A): now also K62.2; no longer K62.1
- net at D66.2 (A): now also K66.2; no longer K66.1
- net at D6.2 (A): now also K6.2; no longer K6.1
- net at D85.2 (A): now also K85.2; no longer K85.1
- net at D11.2 (A): now also K11.2; no longer K11.1
- net at D94.2 (A): now also K94.2; no longer K94.1
- net at D25.2 (A): now also K25.2; no longer K25.1
- net at D7.2 (A): now also K7.2; no longer K7.1
- net at D26.2 (A): now also K26.2; no longer K26.1
- net at D51.2 (A): now also K51.2; no longer K51.1
- net at D64.2 (A): now also K64.2; no longer K64.1
- net at D107.2 (A): now also K107.2; no longer K107.1
- net at D86.2 (A): now also K86.2; no longer K86.1
- net at D108.2 (A): now also K108.2; no longer K108.1
- net at D58.2 (A): now also K58.2; no longer K58.1
- net at D78.2 (A): now also K78.2; no longer K78.1
- net at D84.2 (A): now also K84.2; no longer K84.1
- net at D17.2 (A): now also K17.2; no longer K17.1
- net at D16.2 (A): now also K16.2; no longer K16.1
- net at D40.2 (A): now also K40.2; no longer K40.1
- net at D87.2 (A): now also K87.2; no longer K87.1
- net at D59.2 (A): now also K59.2; no longer K59.1
- net at D30.2 (A): now also K30.2; no longer K30.1
- net at D35.2 (A): now also K35.2; no longer K35.1
- net at D12.2 (A): now also K12.2; no longer K12.1
- net at D57.2 (A): now also K57.2; no longer K57.1
- net at D96.2 (A): now also K96.2; no longer K96.1
- net at D65.2 (A): now also K65.2; no longer K65.1
- net at D81.2 (A): now also K81.2; no longer K81.1
- net at D82.2 (A): now also K82.2; no longer K82.1
- net at D50.2 (A): now also K50.2; no longer K50.1
- net at D21.2 (A): now also K21.2; no longer K21.1
- net at D39.2 (A): now also K39.2; no longer K39.1
- net at D67.2 (A): now also K67.2; no longer K67.1
- net at D98.2 (A): now also K98.2; no longer K98.1
- net at D47.2 (A): now also K47.2; no longer K47.1
- net at D15.2 (A): now also K15.2; no longer K15.1
- net at D4.2 (A): now also K4.2; no longer K4.1
- net at D54.2 (A): now also K54.2; no longer K54.1
- net at D80.2 (A): now also K80.2; no longer K80.1
- net at D53.2 (A): now also K53.2; no longer K53.1
- net at D27.2 (A): now also K27.2; no longer K27.1
- net at D41.2 (A): now also K41.2; no longer K41.1
- net at D44.2 (A): now also K44.2; no longer K44.1
- net at D13.2 (A): now also K13.2; no longer K13.1
- net at D90.2 (A): now also K90.2; no longer K90.1
- net at D106.2 (A): now also K106.2; no longer K106.1
- net at D10.2 (A): now also K10.2; no longer K10.1
- net at D33.2 (A): now also K33.2; no longer K33.1
- net at D97.2 (A): now also K97.2; no longer K97.1
- net at D23.2 (A): now also K23.2; no longer K23.1
- net at D20.2 (A): now also K20.2; no longer K20.1
- net at D103.2 (A): now also K103.2; no longer K103.1
- net at D69.2 (A): now also K69.2; no longer K69.1
- net at D102.2 (A): now also K102.2; no longer K102.1
- net at D34.2 (A): now also K34.2; no longer K34.1
- net at D49.2 (A): now also K49.2; no longer K49.1
- net at D45.2 (A): now also K45.2; no longer K45.1
- net at D24.2 (A): now also K24.2; no longer K24.1
- net at D14.2 (A): now also K14.2; no longer K14.1
- net at D56.2 (A): now also K56.2; no longer K56.1
- net at D74.2 (A): now also K74.2; no longer K74.1
- net at D92.2 (A): now also K92.2; no longer K92.1
- net at D55.2 (A): now also K55.2; no longer K55.1
- net at D9.2 (A): now also K9.2; no longer K9.1
- net at D29.2 (A): now also K29.2; no longer K29.1
- net at D18.2 (A): now also K18.2; no longer K18.1
- net at D46.2 (A): now also K46.2; no longer K46.1
- net at D70.2 (A): now also K70.2; no longer K70.1
- net at D36.2 (A): now also K36.2; no longer K36.1
- net at D1.2 (A): now also K1.2; no longer K1.1
- net at D100.2 (A): now also K100.2; no longer K100.1
- net at D77.2 (A): now also K77.2; no longer K77.1
- net at D95.2 (A): now also K95.2; no longer K95.1
- net at D83.2 (A): now also K83.2; no longer K83.1
- net at D79.2 (A): now also K79.2; no longer K79.1
- net at D105.2 (A): now also K105.2; no longer K105.1
- net at D42.2 (A): now also K42.2; no longer K42.1
- net at D31.2 (A): now also K31.2; no longer K31.1
- net at D48.2 (A): now also K48.2; no longer K48.1
- net at D93.2 (A): now also K93.2; no longer K93.1
- net at D104.2 (A): now also K104.2; no longer K104.1
- net at D28.2 (A): now also K28.2; no longer K28.1
- net at D76.2 (A): now also K76.2; no longer K76.1
- net at D88.2 (A): now also K88.2; no longer K88.1
- net at D22.2 (A): now also K22.2; no longer K22.1
- net at D37.2 (A): now also K37.2; no longer K37.1
- net at D2.2 (A): now also K2.2; no longer K2.1
- net at D72.2 (A): now also K72.2; no longer K72.1
- net at D32.2 (A): now also K32.2; no longer K32.1
- net at D19.2 (A): now also K19.2; no longer K19.1
- net at D73.2 (A): now also K73.2; no longer K73.1
- net at D52.2 (A): now also K52.2; no longer K52.1
- net at D68.2 (A): now also K68.2; no longer K68.1
- net at D43.2 (A): now also K43.2; no longer K43.1
- net at D60.2 (A): now also K60.2; no longer K60.1
- net at D61.2 (A): now also K61.2; no longer K61.1
- net at D5.2 (A): now also K5.2; no longer K5.1
