File: Duet-Plate/Duet-Switch-Tester.kicad_pcb (KiCad board)
At the start: 2 copper layers, 392.7 x 128.9 mm, 19 parts

Commit message: Make case parts prettier
Parts:
- removed the G*** at (414.3, 153.6)
- added G***: LOGO, locallib:ai-4.8-mask, F.Cu at (414.3, 153.6)
Routing:
- added copper zone on B.Cu, net (none)
- added copper zone on F.Cu, net (none)

Commit message: Generate production data
Parts:
- removed G***: LOGO, locallib:ai-4.8-mask
Other:
- board text removed: "DUET"
- board text removed: "Switch Tester"
